Commit message: udacity_bot replaced

File: src/slam_project/urdf/slam_bot.xacro (robot description, xacro)
@@ -157,5 +157,5 @@
       <origin xyz="0 0 0" rpy=" 0 0 0"/>
       <geometry>
-        <mesh filename="package://udacity_bot/meshes/hokuyo.dae"/>
+        <mesh filename="package://slam_project/meshes/hokuyo.dae"/>
       </geometry>
     </visual>

Commit message: xacro camera rgbd definition

File: src/slam_project/urdf/slam_bot.xacro (robot description, xacro)
@@ -142,4 +142,10 @@
     <parent link="chassis"/>
   </joint>
+  <link name="camera_rgbd_frame"></link>
+  <joint name="camera_rgbd_joint" type="fixed">
+    <origin xyz="0 0 0" rpy="-${pi/2} 0 -${pi/2}"/>
+    <parent link="camera"/>
+    <child link="camera_rgbd_frame"/>
+  </joint>
   <link name='hokuyo'>
     <inertial>
